Commit message: Added camera frame

File: robots/tiago_dual.urdf.xacro (robot description, xacro)
@@ -7,3 +7,9 @@
     <child link="base_footprint"/>
 </joint>
+<link name="camera_right_frame"/>
+<joint name="camera_right_frame_joint" type="fixed">
+    <origin rpy="1.57079632679 0 0" xyz="0.072 -0.085 0.0"/>
+    <parent link="wrist_right_ft_tool_link"/>
+    <child link="camera_right_frame"/>
+</joint>
 </robot>

Commit message: Adjysted right camera tf

File: robots/tiago_dual.urdf.xacro (robot description, xacro)
@@ -9,5 +9,5 @@
 <link name="camera_right_frame"/>
 <joint name="camera_right_frame_joint" type="fixed">
-    <origin rpy="1.57079632679 0 0" xyz="0.072 -0.085 0.0"/>
+    <origin rpy="1.57079632679 0 0" xyz="0.072 -0.085 -0.032"/>
     <parent link="wrist_right_ft_tool_link"/>
     <child link="camera_right_frame"/>

Commit message: Update camera_right_frame

File: robots/tiago_dual.urdf.xacro (robot description, xacro)
@@ -9,5 +9,5 @@
 <link name="camera_right_frame"/>
 <joint name="camera_right_frame_joint" type="fixed">
-    <origin rpy="1.57079632679 0 0" xyz="0.072 -0.085 -0.032"/>
+    <origin rpy="1.57079632679 0 0" xyz="1.072 -0.085 -0.032"/>
     <parent link="wrist_right_ft_tool_link"/>
     <child link="camera_right_frame"/>

Commit message: Added camera_left_frame

File: robots/tiago_dual.urdf.xacro (robot description, xacro)
@@ -13,3 +13,9 @@
     <child link="camera_right_frame"/>
 </joint>
+<link name="camera_left_frame"/>
+<joint name="camera_left_frame_joint" type="fixed">
+    <origin rpy="1.57079632679 0 0" xyz="1.072 -0.085 -0.032"/>
+    <parent link="wrist_left_ft_tool_link"/>
+    <child link="camera_left_frame"/>
+</joint>
 </robot>

Commit message: Added head camera frame

File: robots/tiago_dual.urdf.xacro (robot description, xacro)
@@ -19,3 +19,9 @@
     <child link="camera_left_frame"/>
 </joint>
+<link name="camera_head_frame"/>
+<joint name="camera_head_frame_joint" type="fixed">
+    <origin rpy="3.093 0.759 -0.027" xyz="0.127 0.031 1.174"/>
+    <parent link="base_link"/>
+    <child link="camera_head_frame"/>
+</joint>
 </robot>

Commit message: Changed camera_head_frame transformation

File: robots/tiago_dual.urdf.xacro (robot description, xacro)
@@ -21,5 +21,5 @@
 <link name="camera_head_frame"/>
 <joint name="camera_head_frame_joint" type="fixed">
-    <origin rpy="3.093 0.759 -0.027" xyz="0.127 0.031 1.174"/>
+    <origin rpy="-3.1415927 0.0 0.0" xyz="0.171591 0.0112369 1.20358"/>
     <parent link="base_link"/>
     <child link="camera_head_frame"/>
